File: iocon.kicad_sch (KiCad schematic)
At the start: 2 parts, among them J1 Conn_02x13_Odd_Even, J2 Conn_01x03

Commit message: set U3+U4 voltage to ~2.7V
Parts:
- renumbered J1 to J3, J2 to J4
Changed lines of the file:
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@@
 		(dnp no)
 		(fields_autoplaced yes)
-		(property "Reference" "J2"
+		(property "Reference" "J4"
 			(at 147.32 96.5199 0)
 			(effects
@@
 		(dnp no)
 		(fields_autoplaced yes)
-		(property "Reference" "J1"
+		(property "Reference" "J3"
 			(at 120.65 60.96 0)
 			(effects
